File: hardware/scuznet.sch (KiCad schematic (older format))
At the start: 93 parts, among them J1 SCSI, J2 Barrel_Jack_2P, J3 RJ45-TRANSFO, J4 Micro_SD_Card, J5 PDI, J6 HS, J7 HS, U1 ATXMEGA128A3U, U10 LM1117-ADJ, U2 74LVTH126, U3 74LVTH126, U4 74LVTH126, U5 74LVTH126, U6 74LVC14, U7 74LVTH574, U8 ENC28J60-I/SP, U9 MCP1826S, Y1 25MHz

Commit message: Hardware revision 2.
Parts:
- removed J1: SCSI, scuznet:D25S13A, symbol DB25_Female
- removed J4: Micro_SD_Card, scuznet:0472192001, symbol Micro_SD_Card
- removed J6, J7: HS, Heatsinks:Heatsink_AAVID_573300D00010G_TO-263, symbol Conn_01x01
- removed R18: 3K3, Capacitors_SMD:C_0603, symbol R
- removed U7: 74LVTH574, Housings_SOIC:SOIC-20W_7.5x12.8mm_Pitch1.27mm, symbol 74LS574
- added D4: LED, LED_SMD:LED_0805_2012Metric, symbol Device:LED
- added D5: SP0502BAHT, Package_TO_SOT_SMD:SOT-23, symbol Power_Protection:SP0502BAHT
- added J1: SCSI, scuznet:D25S13A, symbol Connector:DB25_Female_MountingHoles
- added J4: SD_Card, Connector_Card:SD_Kyocera_145638009211859+, symbol Connector:SD_Card
- added J6: USB_B_Micro, Connector_USB:USB_Micro-B_Wuerth_629105150521_CircularHoles, symbol Connector:USB_B_Micro
- added R15: 165, Resistor_SMD:R_0603_1608Metric, symbol Device:R
- added R5, R6: 10K, Resistor_SMD:R_0603_1608Metric, symbol Device:R
- added unit 5 of U2
- added unit 5 of U3
- added unit 5 of U4
- added unit 5 of U5
- added unit 7 of U6
- added U7: 74LVTH245, Package_SO:SOIC-20W_7.5x12.8mm_P1.27mm, symbol 74xx:74LS245
- C1: footprint Capacitors_THT:CP_Radial_D6.3mm_P2.50mm -> Capacitor_THT:CP_Radial_D6.3mm_P2.50mm; symbol CP1 -> Device:CP1
- C10, C11, C12, C13, C14, C15, C16, C17, C18, C19, C20, C21, C23, C24, C25, C26, C27, C28, C29, C30, C31, C32, C40, C41: footprint Capacitors_SMD:C_0603 -> Capacitor_SMD:C_0603_1608Metric; symbol C -> Device:C
- C2, C3, C4, C5, C6, C7: footprint Capacitors_SMD:C_0805 -> Capacitor_SMD:C_0805_2012Metric; symbol C -> Device:C
- D1: footprint Diodes_SMD:D_SMB -> Diode_SMD:D_SMB; symbol D -> Device:D
- D2, D3: footprint LEDs:LED_0805 -> LED_SMD:LED_0805_2012Metric; symbol LED -> Device:LED
- F1: footprint Fuse_Holders_and_Fuses:Fuse_SMD1206_Wave -> Fuse:Fuse_1206_3216Metric_Pad1.42x1.75mm_HandSolder; symbol Fuse -> Device:Fuse
- J2: symbol Barrel_Jack_2P -> scuznet:Barrel_Jack_2P
- J3: footprint scuznet:SI-60062-F -> Connector_RJ:RJ45_Amphenol_RJMG1BD3B8K1ANR; symbol RJ45-TRANSFO -> Connector:RJ45_Amphenol_RJMG1BD3B8K1ANR
- J5: footprint Connectors:IDC_Header_Straight_6pins -> Connector_PinHeader_2.54mm:PinHeader_2x03_P2.54mm_Vertical; symbol Conn_02x03_Odd_Even -> Connector_Generic:Conn_02x03_Odd_Even
- L1: footprint Capacitors_SMD:C_0603 -> Capacitor_SMD:C_0603_1608Metric; symbol Ferrite_Bead -> Device:Ferrite_Bead
- R1, R2, R22, R23, R24, R25, R26, R27, R28, R29, R3, R30, R31, R4: footprint Capacitors_SMD:C_0603 -> Resistor_SMD:R_0603_1608Metric; symbol R -> Device:R
- R10: renamed from R9; footprint Capacitors_SMD:C_0603 -> Resistor_SMD:R_0603_1608Metric; symbol R -> Device:R
- R11: renamed from R10; footprint Capacitors_SMD:C_0805 -> Resistor_SMD:R_0603_1608Metric; symbol R -> Device:R
- R12: renamed from R11; footprint Capacitors_SMD:C_0805 -> Resistor_SMD:R_0603_1608Metric; symbol R -> Device:R
- R13: renamed from R12; footprint Capacitors_SMD:C_0805 -> Resistor_SMD:R_0603_1608Metric; symbol R -> Device:R
- R14: renamed from R13; footprint Capacitors_SMD:C_0805 -> Resistor_SMD:R_0603_1608Metric; symbol R -> Device:R
- R16: renamed from R14; footprint Capacitors_SMD:C_0603 -> Resistor_SMD:R_0603_1608Metric; symbol R -> Device:R
- R17: renamed from R15; footprint Capacitors_SMD:C_0603 -> Resistor_SMD:R_0603_1608Metric; symbol R -> Device:R
- R18: renamed from R16; footprint Capacitors_SMD:C_0603 -> Resistor_SMD:R_0603_1608Metric; symbol R -> Device:R
- R19: renamed from R17; footprint Capacitors_SMD:C_0603 -> Resistor_SMD:R_0603_1608Metric; symbol R -> Device:R
- R20, R21: footprint Capacitors_SMD:C_0805 -> Resistor_SMD:R_0603_1608Metric; symbol R -> Device:R
- R32: renamed from R33; footprint Capacitors_SMD:C_0603 -> Resistor_SMD:R_0603_1608Metric; symbol R -> Device:R
- R33: renamed from R34; footprint Capacitors_SMD:C_0603 -> Resistor_SMD:R_0603_1608Metric; symbol R -> Device:R
- R34: renamed from R35; footprint Capacitors_SMD:C_0603 -> Resistor_SMD:R_0603_1608Metric; symbol R -> Device:R
- R35: renamed from R36; footprint Capacitors_SMD:C_0603 -> Resistor_SMD:R_0603_1608Metric; symbol R -> Device:R
- R36: renamed from R37; footprint Capacitors_SMD:C_0603 -> Resistor_SMD:R_0603_1608Metric; symbol R -> Device:R
- R37: renamed from R19; footprint Capacitors_SMD:C_0603 -> Resistor_SMD:R_0603_1608Metric; symbol R -> Device:R
- R7: renamed from R6; footprint Capacitors_SMD:C_0603 -> Resistor_SMD:R_0603_1608Metric; symbol R -> Device:R
- R8: renamed from R7; footprint Capacitors_SMD:C_0603 -> Resistor_SMD:R_0603_1608Metric; symbol R -> Device:R
- R9: renamed from R8; footprint Capacitors_SMD:C_0603 -> Resistor_SMD:R_0603_1608Metric; symbol R -> Device:R
- RN1, RN2: footprint Resistors_THT:R_Array_SIP10 -> Resistor_THT:R_Array_SIP10; symbol R_Network09 -> Device:R_Network09
- TP1, TP2: footprint Connectors_TestPoints:Test_Point_Keystone_5000-5004_Miniature -> TestPoint:TestPoint_Keystone_5000-5004_Miniature; symbol TEST -> Connector:TestPoint
- U1: value ATXMEGA128A3U -> ATXMEGA64A3U; footprint Housings_QFP:TQFP-64_14x14mm_Pitch0.8mm -> Package_QFP:TQFP-64_14x14mm_P0.8mm; symbol ATXMEGA128A3U-AU -> MCU_Microchip_ATmega:ATxmega64A3U-AU
- U10: footprint TO_SOT_Packages_SMD:TO-263-3_TabPin2 -> Package_TO_SOT_THT:TO-220F-3_Horizontal_TabDown; symbol LM1117-ADJ -> Regulator_Linear:LM1117-ADJ
- U2, U3, U4, U5: footprint Housings_SOIC:SOIC-14_3.9x8.7mm_Pitch1.27mm -> Package_SO:SOIC-14_3.9x8.7mm_P1.27mm; symbol 74LS126 -> 74xx:74LS126
- U6: footprint Housings_SOIC:SOIC-14_3.9x8.7mm_Pitch1.27mm -> Package_SO:SOIC-14_3.9x8.7mm_P1.27mm; symbol 74LS14 -> 74xx:74LS14
- U8: footprint Housings_SOIC:SOIC-28W_7.5x17.9mm_Pitch1.27mm -> Package_SO:SOIC-28W_7.5x17.9mm_P1.27mm; symbol ENC28J60-I/SP -> Interface_Ethernet:ENC28J60x-SO
- U9: footprint TO_SOT_Packages_SMD:TO-263-3_TabPin2 -> Package_TO_SOT_SMD:SOT-223-3_TabPin2; symbol MCP1826S -> Regulator_Linear:MCP1826S
- Y1: footprint Crystals:Crystal_HC49-U_Vertical -> Crystal:Crystal_HC49-4H_Vertical; symbol Crystal -> Device:Crystal
Connections:
- net labels added: LED1, LED2
- net labels removed: DCLK, LED
- wire segments 458 -> 573
- no-connect marks 17 -> 18

Commit message: Add files via upload
Parts:
- removed C28, C29: 100nF, Capacitor_SMD:C_0603_1608Metric, symbol Device:C
- removed C40, C41: 27pF, Capacitor_SMD:C_0603_1608Metric, symbol Device:C
- removed C6: 10uF, Capacitor_SMD:C_0805_2012Metric, symbol Device:C
- removed D2, D3, D4: LED, LED_SMD:LED_0805_2012Metric, symbol Device:LED
- removed J1: SCSI, scuznet:D25S13A, symbol Connector:DB25_Female_MountingHoles
- removed J2: Barrel_Jack_2P, scuznet:PJ-037A, symbol scuznet:Barrel_Jack_2P
- removed J3: RJ45-TRANSFO, Connector_RJ:RJ45_Amphenol_RJMG1BD3B8K1ANR, symbol Connector:RJ45_Amphenol_RJMG1BD3B8K1ANR
- removed L1: Ferrite_Bead, Capacitor_SMD:C_0603_1608Metric, symbol Device:Ferrite_Bead
- removed R10: 2K32, Resistor_SMD:R_0603_1608Metric, symbol Device:R
- removed R11, R12, R13: 330, Resistor_SMD:R_0603_1608Metric, symbol Device:R
- removed R16, R17, R18, R19: 49.9, Resistor_SMD:R_0603_1608Metric, symbol Device:R
- removed R3, R4: 10K, Resistor_SMD:R_0603_1608Metric, symbol Device:R
- removed R9: 22, Resistor_SMD:R_0603_1608Metric, symbol Device:R
- removed U8: ENC28J60-I/SP, Package_SO:SOIC-28W_7.5x17.9mm_P1.27mm, symbol Interface_Ethernet:ENC28J60x-SO
- removed Y1: 25MHz, Crystal:Crystal_HC49-4H_Vertical, symbol Device:Crystal
- added J1: 50PinSCSI, Connector_PinHeader_2.00mm:PinHeader_2x25_P2.00mm_Vertical, symbol scuznet-rescue:50PinSCSI-50pinscsi
- added J2: Conn_02x05_Odd_Even_SPI, Connector_PinHeader_2.54mm:PinHeader_2x05_P2.54mm_Vertical, symbol scuznet:Conn_02x05_Odd_Even_SPI
- added JLED_1, JLED_2: Conn_01x02, scuznet:2pin, symbol scuznet:Conn_01x02
- C1: symbol Device:CP1 -> scuznet-rescue:CP1-Device
- C10, C11, C12, C13, C14, C15, C16, C17, C18, C19, C2, C20, C21, C23, C24, C25, C26, C27, C3, C30, C31, C32, C4, C5, C7: symbol Device:C -> scuznet-rescue:C-Device
- D1: symbol Device:D -> scuznet-rescue:D-Device
- D5: symbol Power_Protection:SP0502BAHT -> scuznet-rescue:SP0502BAHT-Power_Protection
- F1: symbol Device:Fuse -> scuznet-rescue:Fuse-Device
- J4: symbol Connector:SD_Card -> scuznet-rescue:SD_Card-Connector
- J6: symbol Connector:USB_B_Micro -> scuznet-rescue:USB_B_Micro-Connector
- R1, R14, R15, R2, R20, R21, R22, R23, R24, R25, R26, R27, R28, R29, R30, R31, R32, R33, R34, R35, R36, R37, R5, R6, R7, R8: symbol Device:R -> scuznet-rescue:R-Device
- RN1, RN2: symbol Device:R_Network09 -> scuznet-rescue:R_Network09-Device
- TP1, TP2: symbol Connector:TestPoint -> scuznet-rescue:TestPoint-Connector
- U1: symbol MCU_Microchip_ATmega:ATxmega64A3U-AU -> scuznet-rescue:ATxmega64A3U-AU-MCU_Microchip_ATmega
- U10: symbol Regulator_Linear:LM1117-ADJ -> scuznet-rescue:LM1117-ADJ-Regulator_Linear
- U2, U3, U4, U5: symbol 74xx:74LS126 -> scuznet-rescue:74LS126-74xx
- U6: symbol 74xx:74LS14 -> scuznet-rescue:74LS14-74xx
- U7: symbol 74xx:74LS245 -> scuznet-rescue:74LS245-74xx
- U9: symbol Regulator_Linear:MCP1826S -> scuznet-rescue:MCP1826S-Regulator_Linear
Connections:
- net labels removed: LEDA, LEDB, TPIN+, TPIN-, TPOUT+, TPOUT-
- wire segments 573 -> 490
- no-connect marks 18 -> 17
